File: Analog.kicad_sch (KiCad schematic)
At the start: 6 parts

Commit message: Updated with recent progress on schematic capture
Parts:
- renumbered C1 to C31, C2 to C32, R1 to R23, R2 to R24, R3 to R25, R4 to R26
Changed lines of the file:
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@@
 	(generator "eeschema")
 	(generator_version "8.0")
-	(paper "A4")
+	(paper "A")
 	(title_block
 		(date "mar. 31 mars 2015")
@@
 		(dnp no)
 		(fields_autoplaced yes)
-		(property "Reference" "R1"
+		(property "Reference" "R23"
 			(at 135.89 66.0399 0)
 			(effects
@@
 		(pin "2"
 		)
-		(instances
-			(project "stereo-hub"
-				(path "/e63e39d7-6ac0-4ffd-8aa3-1841a4541b55/21a9ada9-ea3e-4ac7-897f-beb15c972456"
-					(reference "R1")
-					(unit 1)
-				)
-			)
-		)
 	)
 	(symbol
@@
 		(dnp no)
 		(fields_autoplaced yes)
-		(property "Reference" "R3"
+		(property "Reference" "R25"
 			(at 146.05 68.58 90)
 			(effects
@@
 		(pin "2"
 		)
-		(instances
-			(project "stereo-hub"
-				(path "/e63e39d7-6ac0-4ffd-8aa3-1841a4541b55/21a9ada9-ea3e-4ac7-897f-beb15c972456"
-					(reference "R3")
-					(unit 1)
-				)
-			)
-		)
 	)
 	(symbol
@@
 		(dnp no)
 		(fields_autoplaced yes)
-		(property "Reference" "C1"
+		(property "Reference" "C31"
 			(at 157.48 81.2799 0)
 			(effects
@@
 		(pin "2"
 		)
-		(instances
-			(project "stereo-hub"
-				(path "/e63e39d7-6ac0-4ffd-8aa3-1841a4541b55/21a9ada9-ea3e-4ac7-897f-beb15c972456"
-					(reference "C1")
-					(unit 1)
-				)
-			)
-		)
 	)
 	(symbol
@@
 		(dnp no)
 		(fields_autoplaced yes)
-		(property "Reference" "#PWR03"
+		(property "Reference" "#PWR071"
 			(at 153.67 95.25 0)
 			(effects
@@
 		(pin "1"
 		)
-		(instances
-			(project "stereo-hub"
-				(path "/e63e39d7-6ac0-4ffd-8aa3-1841a4541b55/21a9ada9-ea3e-4ac7-897f-beb15c972456"
-					(reference "#PWR03")
-					(unit 1)
-				)
-			)
-		)
 	)
 	(symbol
@@
 		(dnp no)
 		(fields_autoplaced yes)
-		(property "Reference" "#PWR04"
+		(property "Reference" "#PWR072"
 			(at 153.67 134.62 0)
 			(effects
@@
 		(pin "1"
 		)
-		(instances
-			(project "stereo-hub"
-				(path "/e63e39d7-6ac0-4ffd-8aa3-1841a4541b55/21a9ada9-ea3e-4ac7-897f-beb15c972456"
-					(reference "#PWR04")
-					(unit 1)
-				)
-			)
-		)
 	)
 	(symbol
@@
 		(dnp no)
 		(fields_autoplaced yes)
-		(property "Reference" "R4"
+		(property "Reference" "R26"
 			(at 146.05 107.95 90)
 			(effects
@@
 		(pin "2"
 		)
-		(instances
-			(project "stereo-hub"
-				(path "/e63e39d7-6ac0-4ffd-8aa3-1841a4541b55/21a9ada9-ea3e-4ac7-897f-beb15c972456"
-					(reference "R4")
-					(unit 1)
-				)
-			)
-		)
 	)
 	(symbol
@@
 		(dnp no)
 		(fields_autoplaced yes)
-		(property "Reference" "C2"
+		(property "Reference" "C32"
 			(at 157.48 120.6499 0)
 			(effects
@@
 		(pin "2"
 		)
-		(instances
-			(project "stereo-hub"
-				(path "/e63e39d7-6ac0-4ffd-8aa3-1841a4541b55/21a9ada9-ea3e-4ac7-897f-beb15c972456"
-					(reference "C2")
-					(unit 1)
-				)
-			)
-		)
 	)
 	(symbol
@@
 		(dnp no)
 		(fields_autoplaced yes)
-		(property "Reference" "#PWR02"
+		(property "Reference" "#PWR070"
 			(at 133.35 104.14 0)
 			(effects
@@
 		(pin "1"
 		)
-		(instances
-			(project "stereo-hub"
-				(path "/e63e39d7-6ac0-4ffd-8aa3-1841a4541b55/21a9ada9-ea3e-4ac7-897f-beb15c972456"
-					(reference "#PWR02")
-					(unit 1)
-				)
-			)
-		)
 	)
 	(symbol
@@
 		(dnp no)
 		(fields_autoplaced yes)
-		(property "Reference" "#PWR01"
+		(property "Reference" "#PWR069"
 			(at 133.35 64.77 0)
 			(effects
@@
 		(pin "1"
 		)
-		(instances
-			(project "stereo-hub"
-				(path "/e63e39d7-6ac0-4ffd-8aa3-1841a4541b55/21a9ada9-ea3e-4ac7-897f-beb15c972456"
-					(reference "#PWR01")
-					(unit 1)
-				)
-			)
-		)
 	)
 	(symbol
@@
 		(dnp no)
 		(fields_autoplaced yes)
-		(property "Reference" "R2"
+		(property "Reference" "R24"
 			(at 135.89 105.4099 0)
 			(effects
@@
 		(pin "2"
 		)
-		(instances
-			(project "stereo-hub"
-				(path "/e63e39d7-6ac0-4ffd-8aa3-1841a4541b55/21a9ada9-ea3e-4ac7-897f-beb15c972456"
-					(reference "R2")
-					(unit 1)
-				)
-			)
-		)
-	)
+	)
