File: CAN.kicad_sch (KiCad schematic)
At the start: 7 parts, among them U3 MCP2542FDxMF

Commit message: Updated with recent progress on schematic capture
Parts:
- removed C23, C26: 0.1uF, symbol Device:C
- removed C24: 1uF, symbol Device:C
- removed C25: 10uF, symbol Device:C
- removed R21: 120r, symbol Device:R_US
- removed R6: 4.7k, symbol Device:R_US
- removed U3: MCP2542FDxMF, Package_DFN_QFN:DFN-8-1EP_3x3mm_P0.65mm_EP1.55x2.4mm, symbol Interface_CAN_LIN:MCP2542FDxMF
- added C1, C2: 10uF, symbol Device:C_Small
- added C37, C38: 0.1uF, symbol Device:C_Small
- added J11: DE9_Receptacle, symbol Connector:DE9_Receptacle
- added R1: 120r, symbol Device:R_US
- added U8: ISO1044BD, Package_SO:SOIC-8_3.9x4.9mm_P1.27mm, symbol Interface_CAN_LIN:ISO1044BD
- added U9: LM1117MP-5.0, Package_TO_SOT_SMD:SOT-223-3_TabPin2, symbol Regulator_Linear:LM1117MP-5.0
Connections:
- net +3.3V: now also C38.1, U8.1 (VCC1)
- net D+: now also J11.7, R1.1, U8.6 (CANH)
- net D-: now also J11.2, R1.2, U8.5 (CANL)
- net GND: now also C38.2, U8.4 (GND1)
- net RXD: now also U8.3 (RXD)
- net TXD: now also U8.2 (TXD)
- new net: C1.1, J11.9, U9.3 (VI)
- new net: C1.2, C2.2, C37.2, J11.3, U8.7 (GND2), U9.1 (GND)
- new net ISOL-5V: C2.1, C37.1, U8.8 (VCC2), U9.2 (VO)
Other:
- note removed: "Truck CAN Interface/Sniffer"
