File: RaspberryPi.kicad_sch (KiCad schematic)
At the start: 2 parts, among them J1 Raspberry_Pi_2_3, U7 CAT24C128

Commit message: Updated with recent progress on schematic capture
Parts:
- added C12: 0.22uF, Capacitor_SMD:C_0603_1608Metric, symbol Device:C_Small
- added C36: 0.1uF, symbol Device:C
- added D1: BLUE, LED_SMD:LED_0603_1608Metric, symbol Device:LED_Filled
- added J3: 5V 5A Step-down, symbol Connector_Generic:Conn_01x05
- added JP1: WP, symbol Jumper:SolderJumper_2_Bridged
- added R17: 470r, Resistor_SMD:R_0603_1608Metric, symbol Device:R_US
- added R19, R26, R27, R28: 3.9k, symbol Device:R_US
- added R29: 1k, symbol Device:R_US
- U7: value CAT24C128 -> CAT24C32
Connections:
- net +3.3V: now also C36.1, R19.1, R26.1, R27.1, R28.1, R29.1
- net +5V: now also D1.2 (A), J3.5 (Pin_5)
- net GND: now also U7.1 (A0), U7.2 (A1), U7.3 (A2), C12.2, C36.2, J3.3 (Pin_3), J3.4 (Pin_4), JP1.1 (A), R17.2
- net SCL: now also R27.2
- net SDA: now also R28.2
- net at J1.27 (ID_SD/GPIO0), U7.5 (SDA): now also R19.2
- net at J1.28 (ID_SC/GPIO1), U7.6 (SCL): now also R26.2
- net at U7.7 (WP): now also JP1.2 (B), R29.2
- new net: D1.1 (K), R17.1
- new net +24V: C12.1, J3.2 (Pin_2)
- no-connect marks 0 -> 25
Other:
- note added: "Cut this jumper to write- protect the EEPROM"
- moved on the sheet: J1, U7
